File: electronics/fuente_regulable/fuente_regulable.kicad_sch (KiCad schematic)
At the start: 62 parts, among them J1 HDR-3x1, J2 VIN, J3 ON OFF, J4 VIN, J5 HDR-4x1, J6 HDR-5x1, J7 HDR-4x1, J8 HDR-4x1, P1 USB_C_Plug_USB2.0, Q1 Q_NMOS_Depletion_GDS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

Commit message: adding files to repo
Other:
- note added: "Generic 3.3 I2C"
- note added: "Input voltaje : 12V Output voltaje: 25 to 100V"
- note added: "Interface"
- note added: "LCD 5V I2C"
- note added: "Power IN Regs"
- note added: "Rotary encoder"
- note removed: "Input voltaje : 5V to 12V Output voltaje: 25 to 100V"
- note removed: "Power IN"
- moved on the sheet: C10, C11, C12, C13, C14, C15, C16, C17, C6, C7, C8, C9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
